File: full_project.sch (KiCad schematic (older format))
At the start: 36 parts, among them J1 Conn_01x16, J12 V_OFFSET, J14 Conn_01x02, J2 Raspberry_Pi_2_3, J3 Conn_01x08, J4 Screw_Terminal_01x04_titrator, J5 RF_Shield_Two_Pieces, J6 BNC_Jack, J8 Screw_Terminal_01x03, Q1 PN2222A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

Commit message: Silkscreening and most final adjustments done
Parts:
- added H1, H2, H3, H4: MountingHole, MountingHole:MountingHole_3mm, symbol Mechanical:MountingHole
Connections:
- wire segments 176 -> 175
Other:
- note added: "Raspberry Pi Mounting Holes\n(Non-Plated Through Holes)"
- note removed: "Absolute Max Rating For Analog Input to Ground: \n 10mA continuous, -0.3 to VDD + 0.3V \nAnalog Input Voltage: +/- \n\nNot suited for 12V max output from \nop amps in original design."
Changed lines of the file:
@@
 encoding utf-8
 Sheet 1 1
-Title "Automated Alkalinity Titrator"
-Date "2021-02-04"
-Rev "1.3"
+Title "WWU Alkalinity Titrator"
+Date "2021-03-07"
+Rev "2.0"
 Comp "Open Ocean Project"
 Comment1 "Original Designer: Greg Birge"
@@
 Wire Notes Line
 	1725 6375 2125 6375
-Text Notes 700  1100 0    50   ~ 0
-Absolute Max Rating For Analog Input to Ground: \n        10mA continuous, -0.3 to VDD + 0.3V \nAnalog Input Voltage: +/- \n\nNot suited for 12V max output from \nop amps in original design.
-Wire Notes Line
-	675  600  675  1125
-Wire Notes Line
-	675  1125 2750 1125
-Wire Notes Line
-	2750 1125 2750 600
-Wire Notes Line
-	2750 600  675  600
 NoConn ~ 2600 3500
 Text Notes 8225 4900 0    50   ~ 0
@@
 Wire Wire Line
 	6550 2775 6550 2900
-Connection ~ 5725 2775
-Wire Wire Line
-	5725 2775 5725 2925
 Wire Wire Line
 	5725 2475 5725 2775
@@
 	5175 7525 5375 7525
 Text Label 4950 3000 0    50   ~ 0
-PSU_AGND
-Text Label 5725 2925 0    50   ~ 0
 PSU_AGND
 Text Label 5975 4200 0    50   ~ 0
@@
 NoConn ~ 10025 4850
 NoConn ~ 10025 4750
+$Comp
+L Mechanical:MountingHole H3
+U 1 1 604FB748
+P 1350 700
+F 0 "H3" H 1450 746 50  0000 L CNN
+F 1 "MountingHole" H 1450 655 50  0000 L CNN
+F 2 "MountingHole:MountingHole_3mm" H 1350 700 50  0001 C CNN
+F 3 "~" H 1350 700 50  0001 C CNN
+	1    1350 700
+	1    0    0    -1
+$EndComp
+$Comp
+L Mechanical:MountingHole H4
+U 1 1 604FC2A5
+P 1350 975
+F 0 "H4" H 1450 1021 50  0000 L CNN
+F 1 "MountingHole" H 1450 930 50  0000 L CNN
+F 2 "MountingHole:MountingHole_3mm" H 1350 975 50  0001 C CNN
+F 3 "~" H 1350 975 50  0001 C CNN
+	1    1350 975
+	1    0    0    -1
+$EndComp
+$Comp
+L Mechanical:MountingHole H1
+U 1 1 604FC932
+P 650 700
+F 0 "H1" H 750 746 50  0000 L CNN
+F 1 "MountingHole" H 750 655 50  0000 L CNN
+F 2 "MountingHole:MountingHole_3mm" H 650 700 50  0001 C CNN
+F 3 "~" H 650 700 50  0001 C CNN
+	1    650  700
+	1    0    0    -1
+$EndComp
+$Comp
+L Mechanical:MountingHole H2
+U 1 1 604FE1D9
+P 650 975
+F 0 "H2" H 750 1021 50  0000 L CNN
+F 1 "MountingHole" H 750 930 50  0000 L CNN
+F 2 "MountingHole:MountingHole_3mm" H 650 975 50  0001 C CNN
+F 3 "~" H 650 975 50  0001 C CNN
+	1    650  975
+	1    0    0    -1
+$EndComp
+Wire Notes Line
+	550  550  2050 550
+Wire Notes Line
+	2050 550  2050 1100
+Wire Notes Line
+	2050 1100 550  1100
+Wire Notes Line
+	550  1100 550  550
+Text Notes 700  1275 0    50   ~ 0
+Raspberry Pi Mounting Holes\n(Non-Plated Through Holes)
 $EndSCHEMATC

Commit message: Extended board, added MAX31685 footprint for new mounting style, added 3.5mm audio jacks, cried a little
Parts:
- added J7, J9: SJ-43515TS, Titrator_Footprints:CUI_SJ-43515TS, symbol SJ-43515TS:SJ-43515TS
- U3, U4: footprint Connector_Molex:Molex_SL_171971-0008_1x08_P2.54mm_Vertical -> Titrator_Footprints:MAX31865; symbol titrator:MAX31865_BO -> titrator:MAX31865_FullBO
Connections:
- wire segments 175 -> 190
- no-connect marks 46 -> 47
Other:
- note added: "The RTD Temp Probes WIll Be Connected\nVia 3.5mm (1/8") audio jack"
- note removed: "May want two 3V3 Power Supplies\n* One for Analog (pH Probe)\n* One for Digital (From Raspberry Pi to Everything Else)"
Changed lines of the file:
@@
 L power:+3V3 #PWR07
 U 1 1 5F10DA7E
-P 6100 5225
-F 0 "#PWR07" H 6100 5075 50  0001 C CNN
-F 1 "+3V3" H 6115 5398 50  0000 C CNN
-F 2 "" H 6100 5225 50  0001 C CNN
-F 3 "" H 6100 5225 50  0001 C CNN
-	1    6100 5225
+P 6100 4850
+F 0 "#PWR07" H 6100 4700 50  0001 C CNN
+F 1 "+3V3" H 6115 5023 50  0000 C CNN
+F 2 "" H 6100 4850 50  0001 C CNN
+F 3 "" H 6100 4850 50  0001 C CNN
+	1    6100 4850
 	1    0    0    -1
 $EndComp
@@
 $EndComp
 Wire Wire Line
-	6100 5225 6250 5225
+	6100 4850 6250 4850
 $Comp
 L power:PWR_FLAG #FLG01
@@
 L power:+3V3 #PWR06
 U 1 1 5F1150D9
-P 4300 5225
-F 0 "#PWR06" H 4300 5075 50  0001 C CNN
-F 1 "+3V3" H 4315 5398 50  0000 C CNN
-F 2 "" H 4300 5225 50  0001 C CNN
-F 3 "" H 4300 5225 50  0001 C CNN
-	1    4300 5225
-	1    0    0    -1
-$EndComp
-Wire Wire Line
-	4300 5225 4450 5225
+P 4600 4850
+F 0 "#PWR06" H 4600 4700 50  0001 C CNN
+F 1 "+3V3" H 4615 5023 50  0000 C CNN
+F 2 "" H 4600 4850 50  0001 C CNN
+F 3 "" H 4600 4850 50  0001 C CNN
+	1    4600 4850
+	1    0    0    -1
+$EndComp
+Wire Wire Line
+	4600 4850 4750 4850
 Wire Wire Line
 	2600 3100 2700 3100
@@
 Text Label 2700 4200 0    50   ~ 0
 SCLK
-NoConn ~ 4450 5425
-NoConn ~ 6250 5425
-NoConn ~ 6950 5525
-NoConn ~ 5150 5525
+NoConn ~ 4750 5050
+NoConn ~ 6250 5050
+NoConn ~ 6950 5150
+NoConn ~ 5450 5150
 $Comp
 L power:GND #PWR04
 U 1 1 5F12F9CC
-P 4050 5375
-F 0 "#PWR04" H 4050 5125 50  0001 C CNN
-F 1 "GND" H 4055 5202 50  0000 C CNN
-F 2 "" H 4050 5375 50  0001 C CNN
-F 3 "" H 4050 5375 50  0001 C CNN
-	1    4050 5375
+P 4350 5000
+F 0 "#PWR04" H 4350 4750 50  0001 C CNN
+F 1 "GND" H 4355 4827 50  0000 C CNN
+F 2 "" H 4350 5000 50  0001 C CNN
+F 3 "" H 4350 5000 50  0001 C CNN
+	1    4350 5000
 	-1   0    0    -1
 $EndComp
@@
 L power:GND #PWR05
 U 1 1 5F130D30
-P 5850 5375
-F 0 "#PWR05" H 5850 5125 50  0001 C CNN
-F 1 "GND" H 5855 5202 50  0000 C CNN
-F 2 "" H 5850 5375 50  0001 C CNN
-F 3 "" H 5850 5375 50  0001 C CNN
-	1    5850 5375
+P 5850 5000
+F 0 "#PWR05" H 5850 4750 50  0001 C CNN
+F 1 "GND" H 5855 4827 50  0000 C CNN
+F 2 "" H 5850 5000 50  0001 C CNN
+F 3 "" H 5850 5000 50  0001 C CNN
+	1    5850 5000
 	-1   0    0    -1
 $EndComp
 Wire Wire Line
-	4400 5525 4450 5525
-Wire Wire Line
-	6200 5525 6250 5525
-Text Label 4400 5525 2    50   ~ 0
+	4700 5150 4750 5150
+Wire Wire Line
+	6200 5150 6250 5150
+Text Label 4700 5150 2    50   ~ 0
 SCLK
-Text Label 6200 5525 2    50   ~ 0
+Text Label 6200 5150 2    50   ~ 0
 SCLK
 Wire Wire Line
-	5850 5375 5850 5325
-Wire Wire Line
-	5850 5325 6250 5325
-Wire Wire Line
-	4050 5325 4050 5375
-Wire Wire Line
-	4050 5325 4450 5325
-Wire Wire Line
-	5200 5225 5150 5225
-Wire Wire Line
-	5200 5325 5150 5325
-Wire Wire Line
-	5200 5425 5150 5425
-Wire Wire Line
-	7000 5225 6950 5225
-Wire Wire Line
-	7000 5325 6950 5325
-Wire Wire Line
-	7000 5425 6950 5425
-Text Label 5200 5225 0    50   ~ 0
+	5850 5000 5850 4950
+Wire Wire Line
+	5850 4950 6250 4950
+Wire Wire Line
+	4350 4950 4350 5000
+Wire Wire Line
+	4350 4950 4750 4950
+Wire Wire Line
+	5500 4850 5450 4850
+Wire Wire Line
+	5500 4950 5450 4950
+Wire Wire Line
+	5500 5050 5450 5050
+Wire Wire Line
+	7000 4850 6950 4850
+Wire Wire Line
+	7000 4950 6950 4950
+Wire Wire Line
+	7000 5050 6950 5050
+Text Label 5500 4850 0    50   ~ 0
 MOSI
-Text Label 5200 5325 0    50   ~ 0
+Text Label 5500 4950 0    50   ~ 0
 MISO
-Text Label 5200 5425 0    50   ~ 0
+Text Label 5500 5050 0    50   ~ 0
 CE0
-Text Label 7000 5425 0    50   ~ 0
+Text Label 7000 5050 0    50   ~ 0
 CE1
-Text Label 7000 5225 0    50   ~ 0
+Text Label 7000 4850 0    50   ~ 0
 MOSI
-Text Label 7000 5325 0    50   ~ 0
+Text Label 7000 4950 0    50   ~ 0
 MISO
 Wire Wire Line
@@
 Wire Wire Line
 	1825 6125 1825 6225
-Wire Wire Line
-	2650 4400 2600 4400
 Text Label 2600 4500 0    50   ~ 0
 PWM
@@
 $EndComp
 $Comp
-L titrator:MAX31865_BO U4
+L titrator:MAX31865_FullBO U4
 U 1 1 5F114422
-P 6600 5375
-F 0 "U4" H 6600 5750 50  0000 C CNN
-F 1 "MAX31865_BO" H 6600 5659 50  0000 C CNN
-F 2 "Connector_Molex:Molex_SL_171971-0008_1x08_P2.54mm_Vertical" H 6600 5375 50  0001 C CNN
-F 3 "https://datasheets.maximintegrated.com/en/ds/MAX31865.pdf" H 6600 5375 50  0001 C CNN
-	1    6600 5375
+P 6600 5000
+F 0 "U4" H 6600 5375 50  0000 C CNN
+F 1 "MAX31865_BO" H 6600 5284 50  0000 C CNN
+F 2 "Titrator_Footprints:MAX31865" H 6600 5000 50  0001 C CNN
+F 3 "https://datasheets.maximintegrated.com/en/ds/MAX31865.pdf" H 6600 5000 50  0001 C CNN
+	1    6600 5000
 	1    0    0    -1
 $EndComp
@@
 U 1 1 5F1C81E1
 P 3675 6225
-F 0 "J4" H 3625 6550 50  0000 L CNN
-F 1 "Screw_Terminal_01x04_titrator" H 3600 6425 50  0000 L CNN
+F 0 "J4" H 3625 6450 50  0000 L CNN
+F 1 "Screw_Terminal_01x04_titrator" H 3525 5900 50  0000 L CNN
 F 2 "TerminalBlock:TerminalBlock_bornier-4_P5.08mm" H 3675 6225 50  0001 C CNN
 F 3 "~" H 3675 6225 50  0001 C CNN
@@
 Wire Notes Line
 	1725 6375 2125 6375
-NoConn ~ 2600 3500
 Text Notes 8225 4900 0    50   ~ 0
 Need vigorous stirring\nfor 10min once the pH \nhits 3.5, then goes back \nto a relaxed speed
 NoConn ~ 4850 2675
 NoConn ~ 4850 2775
-Text Notes 575  1925 0    50   ~ 0
-May want two 3V3 Power Supplies\n* One for Analog (pH Probe)\n* One for Digital (From Raspberry Pi to Everything Else)
 Text Notes 2250 5550 0    50   ~ 0
 KEEP AWAY FROM\nANALOG STUFF
@@
 $Comp
 L Amplifier_Operational:LMC6062 U7
-U 2 1 6036177B
-P 4600 4000
-F 0 "U7" H 4600 4367 50  0000 C CNN
-F 1 "LMC662" H 4600 4276 50  0000 C CNN
-F 2 "Package_DIP:DIP-8_W7.62mm" H 4600 4000 50  0001 C CNN
-F 3 "https://www.ti.com/lit/ds/symlink/lmc662.pdf?ts=1612139527764&ref_url=https%253A%252F%252Fwww.google.com%252F" H 4600 4000 50  0001 C CNN
-	2    4600 4000
-	1    0    0    -1
-$EndComp
-$Comp
-L Amplifier_Operational:LMC6062 U7
 U 3 1 603641B9
 P 5950 3425
@@
 NoConn ~ 4300 3900
 NoConn ~ 4300 4100
-NoConn ~ 4900 4000
 Text Notes 4150 4300 0    50   ~ 0
 Second channel of LPF IC
@@
 Text Label 2600 3600 0    50   ~ 0
 KeyRow_2
-Text Label 2650 4400 0    50   ~ 0
+Text Label 2600 3500 0    50   ~ 0
 KeyRow_3
 Text Label 1000 3500 2    50   ~ 0
@@
 	0    1    1    0
 $EndComp
-Text Notes 4675 5725 0    49   ~ 0
+Text Notes 4675 4525 0    49   ~ 0
 CS input initiates and terminates data transfer (enable)
 $Comp
-L titrator:MAX31865_BO U3
+L titrator:MAX31865_FullBO U3
 U 1 1 5F112236
-P 4800 5375
-F 0 "U3" H 4800 5750 50  0000 C CNN
-F 1 "MAX31865_BO" H 4800 5659 50  0000 C CNN
-F 2 "Connector_Molex:Molex_SL_171971-0008_1x08_P2.54mm_Vertical" H 4800 5375 50  0001 C CNN
-F 3 "https://datasheets.maximintegrated.com/en/ds/MAX31865.pdf" H 4800 5375 50  0001 C CNN
-	1    4800 5375
+P 5100 5000
+F 0 "U3" H 5100 5375 50  0000 C CNN
+F 1 "MAX31865_BO" H 5100 5284 50  0000 C CNN
+F 2 "Titrator_Footprints:MAX31865" H 5100 5000 50  0001 C CNN
+F 3 "https://datasheets.maximintegrated.com/en/ds/MAX31865.pdf" H 5100 5000 50  0001 C CNN
+	1    5100 5000
 	1    0    0    -1
 $EndComp
@@
 Text Notes 700  1275 0    50   ~ 0
 Raspberry Pi Mounting Holes\n(Non-Plated Through Holes)
+Wire Wire Line
+	4900 5700 4900 5575
+Wire Wire Line
+	5025 5575 5025 5800
+Wire Wire Line
+	6400 5575 6400 5700
+Wire Wire Line
+	6400 5700 6300 5700
+Wire Wire Line
+	6525 5575 6525 5800
+Wire Wire Line
+	6525 5800 6300 5800
+Wire Wire Line
+	6675 6000 6300 6000
+Wire Wire Line
+	6800 6100 6300 6100
+$Comp
+L SJ-43515TS:SJ-43515TS J7
+U 1 1 6053C631
+P 4350 5900
+F 0 "J7" H 4407 6367 50  0000 C CNN
+F 1 "SJ-43515TS" H 4407 6276 50  0000 C CNN
+F 2 "Titrator_Footprints:CUI_SJ-43515TS" H 4350 5900 50  0001 L BNN
+F 3 "https://www.cuidevices.com/product/resource/sj-4351x.pdf" H 4350 5900 50  0001 L BNN
+F 4 "CUI INC" H 4350 5900 50  0001 L BNN "MANUFACTURER"
+F 5 "MANUFACTURER RECOMMENDATIONS" H 4350 5900 50  0001 L BNN "STANDARD"
+F 6 "1.04" H 4350 5900 50  0001 L BNN "PART_REV"
+	1    4350 5900
+	1    0    0    -1
+$EndComp
+Wire Wire Line
+	5175 5575 5175 6000
+Wire Wire Line
+	4750 6000 5175 6000
+Wire Wire Line
+	5300 5575 5300 6100
+Wire Wire Line
+	4750 6100 5300 6100
+Wire Wire Line
+	4750 5800 5025 5800
+Wire Wire Line
+	4750 5700 4900 5700
+NoConn ~ 4750 5900
+$Comp
+L SJ-43515TS:SJ-43515TS J9
+U 1 1 605A3406
+P 5900 5900
+F 0 "J9" H 5957 6367 50  0000 C CNN
+F 1 "SJ-43515TS" H 5957 6276 50  0000 C CNN
+F 2 "Titrator_Footprints:CUI_SJ-43515TS" H 5900 5900 50  0001 L BNN
+F 3 "https://www.cuidevices.com/product/resource/sj-4351x.pdf" H 5900 5900 50  0001 L BNN
+F 4 "CUI INC" H 5900 5900 50  0001 L BNN "MANUFACTURER"
+F 5 "MANUFACTURER RECOMMENDATIONS" H 5900 5900 50  0001 L BNN "STANDARD"
+F 6 "1.04" H 5900 5900 50  0001 L BNN "PART_REV"
+	1    5900 5900
+	1    0    0    -1
+$EndComp
+Wire Wire Line
+	6675 5575 6675 6000
+Wire Wire Line
+	6800 5575 6800 6100
+NoConn ~ 6300 5900
+Text Notes 4475 6400 0    50   ~ 0
+The RTD Temp Probes WIll Be Connected\nVia 3.5mm (1/8") audio jack
+$Comp
+L power:PWR_FLAG #FLG0103
+U 1 1 605D41A8
+P 5975 4100
+F 0 "#FLG0103" H 5975 4175 50  0001 C CNN
+F 1 "PWR_FLAG" H 5975 4273 50  0000 C CNN
+F 2 "" H 5975 4100 50  0001 C CNN
+F 3 "~" H 5975 4100 50  0001 C CNN
+	1    5975 4100
+	1    0    0    -1
+$EndComp
+NoConn ~ 4900 4000
+$Comp
+L Amplifier_Operational:LMC6062 U7
+U 2 1 6036177B
+P 4600 4000
+F 0 "U7" H 4600 4367 50  0000 C CNN
+F 1 "LMC662" H 4600 4276 50  0000 C CNN
+F 2 "Package_DIP:DIP-8_W7.62mm" H 4600 4000 50  0001 C CNN
+F 3 "https://www.ti.com/lit/ds/symlink/lmc662.pdf?ts=1612139527764&ref_url=https%253A%252F%252Fwww.google.com%252F" H 4600 4000 50  0001 C CNN
+	2    4600 4000
+	1    0    0    -1
+$EndComp
 $EndSCHEMATC

Commit message: not much
Parts:
- added H5, H6: MountingHole, MountingHole:MountingHole_3mm, symbol Mechanical:MountingHole
- added J10: Screw_Terminal_01x02, TerminalBlock:TerminalBlock_bornier-2_P5.08mm, symbol Connector:Screw_Terminal_01x02
Connections:
- net GND: now also J10.2 (Pin_2)
- net at J2.32 (PWM0/GPIO12): now also J10.1 (Pin_1)
Other:
- note added: "SSR (Solid State Relay)"
Changed lines of the file:
@@
 $EndComp
 Wire Notes Line
-	550  550  2050 550
-Wire Notes Line
-	2050 550  2050 1100
-Wire Notes Line
-	2050 1100 550  1100
+	2700 550  2700 1100
 Wire Notes Line
 	550  1100 550  550
@@
 	1    0    0    -1
 $EndComp
+$Comp
+L Mechanical:MountingHole H5
+U 1 1 604871C9
+P 2050 700
+F 0 "H5" H 2150 746 50  0000 L CNN
+F 1 "MountingHole" H 2150 655 50  0000 L CNN
+F 2 "MountingHole:MountingHole_3mm" H 2050 700 50  0001 C CNN
+F 3 "~" H 2050 700 50  0001 C CNN
+	1    2050 700
+	1    0    0    -1
+$EndComp
+$Comp
+L Mechanical:MountingHole H6
+U 1 1 60491872
+P 2050 975
+F 0 "H6" H 2150 1021 50  0000 L CNN
+F 1 "MountingHole" H 2150 930 50  0000 L CNN
+F 2 "MountingHole:MountingHole_3mm" H 2050 975 50  0001 C CNN
+F 3 "~" H 2050 975 50  0001 C CNN
+	1    2050 975
+	1    0    0    -1
+$EndComp
+Wire Notes Line
+	550  550  2700 550
+Wire Notes Line
+	550  1100 2700 1100
+$Comp
+L Connector:Screw_Terminal_01x02 J10
+U 1 1 604B33B0
+P 3175 4400
+F 0 "J10" H 3255 4392 50  0000 L CNN
+F 1 "Screw_Terminal_01x02" H 3255 4301 50  0000 L CNN
+F 2 "TerminalBlock:TerminalBlock_bornier-2_P5.08mm" H 3175 4400 50  0001 C CNN
+F 3 "~" H 3175 4400 50  0001 C CNN
+	1    3175 4400
+	1    0    0    -1
+$EndComp
+Wire Wire Line
+	2600 4400 2975 4400
+$Comp
+L power:GND #PWR016
+U 1 1 604C156D
+P 2975 4500
+F 0 "#PWR016" H 2975 4250 50  0001 C CNN
+F 1 "GND" H 2980 4327 50  0000 C CNN
+F 2 "" H 2975 4500 50  0001 C CNN
+F 3 "" H 2975 4500 50  0001 C CNN
+	1    2975 4500
+	1    0    0    -1
+$EndComp
+Text Notes 3100 4675 0    50   ~ 0
+SSR (Solid State Relay)
 $EndSCHEMATC

Commit message: Please just push
Connections:
- net CE0: now also J2.27 (ID_SD/GPIO0); no longer J2.24 (~CE0~/GPIO8)
- net CE1: now also J2.7 (GCLK0/GPIO4); no longer J2.26 (~CE1~/GPIO7)
Other:
- note added: "IMPORTANT!\nCircuitPython uses CE0 and \nCE1 for chip enable magic. \nDo not use them as chip \nenables! Any other GPIO pin \ncan act as a chip enable \ninstead."
- note added: "TO DO: ADD NEW CHANNEL"
- note added: "TO DO\nHook to 12V"
- note added: "TO DO\nMake this TIP120"
Changed lines of the file:
@@
 Text Label 2700 3200 0    50   ~ 0
 SCL
-Text Label 2700 3800 0    50   ~ 0
+Text Label 2600 3400 0    50   ~ 0
 CE1
-Text Label 2700 3900 0    50   ~ 0
+Text Label 2600 2800 0    50   ~ 0
 CE0
 Text Label 2700 4000 0    50   ~ 0
@@
 Wire Wire Line
 	1400 5000 1400 5100
-$Comp
-L Connector:Raspberry_Pi_2_3 J2
-U 1 1 5F0D7F94
-P 1800 3700
-F 0 "J2" H 1800 4500 50  0000 C CNN
-F 1 "Raspberry_Pi_2_3" H 1800 4400 50  0000 C CNN
-F 2 "Connector_PinSocket_2.54mm:PinSocket_2x20_P2.54mm_Vertical" H 1800 3700 50  0001 C CNN
-F 3 "https://www.raspberrypi.org/documentation/hardware/raspberrypi/schematics/rpi_SCH_3bplus_1p0_reduced.pdf" H 1800 3700 50  0001 C CNN
-	1    1800 3700
-	1    0    0    -1
-$EndComp
-NoConn ~ 2600 3400
+NoConn ~ 2700 3800
 Text Label 7700 5775 2    50   ~ 0
 PWM
@@
 Text Label 1000 3100 2    50   ~ 0
 KeyCol_1
-NoConn ~ 2600 2800
+NoConn ~ 2700 3900
 Text Label 1000 4300 2    50   ~ 0
 KeyCol_2
@@
 Text Notes 3100 4675 0    50   ~ 0
 SSR (Solid State Relay)
+$Comp
+L Connector:Raspberry_Pi_2_3 J2
+U 1 1 5F0D7F94
+P 1800 3700
+F 0 "J2" H 1800 4500 50  0000 C CNN
+F 1 "Raspberry_Pi_2_3" H 1800 4400 50  0000 C CNN
+F 2 "Connector_PinSocket_2.54mm:PinSocket_2x20_P2.54mm_Vertical" H 1800 3700 50  0001 C CNN
+F 3 "https://www.raspberrypi.org/documentation/hardware/raspberrypi/schematics/rpi_SCH_3bplus_1p0_reduced.pdf" H 1800 3700 50  0001 C CNN
+	1    1800 3700
+	1    0    0    -1
+$EndComp
+Text Notes 2975 4125 0    50   ~ 0
+IMPORTANT!\nCircuitPython uses CE0 and \nCE1 for chip enable magic. \nDo not use them as chip \nenables! Any other GPIO pin \ncan act as a chip enable \ninstead.
+Wire Notes Line
+	2750 3800 2950 3800
+Wire Notes Line
+	2750 3900 2850 3900
+Wire Notes Line
+	2850 3900 2850 3800
+Text Notes 8775 5650 0    50   ~ 0
+TO DO\nMake this TIP120
+Text Notes 7700 5050 0    50   ~ 0
+TO DO\nHook to 12V
+Text Notes 4075 3525 0    50   ~ 0
+TO DO: ADD NEW CHANNEL
 $EndSCHEMATC
