File: schematic_for_screenshots.sch (KiCad schematic (older format))
At the start: 45 parts, among them J1 Conn_01x16, J10 Screw_Terminal_01x02, J12 V_OFFSET, J14 Conn_01x02, J2 Raspberry_Pi_2_3, J3 Conn_01x08, J4 Screw_Terminal_01x04_titrator, J5 RF_Shield_Two_Pieces, J6 BNC_Jack, J7 SJ-43515TS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

Commit message: Changed diode footprint
Parts:
- D1: footprint Diode_THT:D_DO-41_SOD81_P10.16mm_Horizontal -> Diode_THT:D_T-1_P12.70mm_Horizontal
Changed lines of the file:
@@
 Gain 8: FS=+/-0.512V -> LSB = 15.625 μV\nGain 16: FS=+/-0.256V -> LSB = 7.812 μV
+$Comp
+L pspice:DIODE D1
+U 1 1 60226A87
+P 8600 5150
+F 0 "D1" H 8600 5415 50  0000 C CNN
+F 1 "DIODE" H 8600 5324 50  0000 C CNN
+F 2 "Diode_THT:D_T-1_P12.70mm_Horizontal" H 8600 5150 50  0001 C CNN
+F 3 "~" H 8600 5150 50  0001 C CNN
+	1    8600 5150
+	0    -1   -1   0
+$EndComp
 $Comp
 L Connector_Generic:Conn_01x02 J14
@@
 $EndComp
 Wire Wire Line
+	8600 4950 8950 4950
+Wire Wire Line
 	9175 4950 9175 5075
+Connection ~ 8600 4950
 Wire Wire Line
 	9175 5175 9175 5350
 Wire Wire Line
 	8600 5350 8600 5575
+Connection ~ 8600 5350
 Wire Wire Line
 	8950 5000 8950 4950
@@
 	1    0    0    -1
 $EndComp
+Wire Wire Line
+	8025 4950 8600 4950
 $Comp
 L Device:R R7
@@
 Wire Notes Line
 	8800 5875 8700 5875
-Connection ~ 8600 5350
-Connection ~ 8600 4950
-Wire Wire Line
-	8025 4950 8600 4950
-Wire Wire Line
-	8600 4950 8950 4950
-$Comp
-L pspice:DIODE D1
-U 1 1 60226A87
-P 8600 5150
-F 0 "D1" H 8600 5415 50  0000 C CNN
-F 1 "DIODE" H 8600 5324 50  0000 C CNN
-F 2 "Diode_THT:D_DO-41_SOD81_P10.16mm_Horizontal" H 8600 5150 50  0001 C CNN
-F 3 "~" H 8600 5150 50  0001 C CNN
-	1    8600 5150
-	0    -1   -1   0
-$EndComp
 $EndSCHEMATC
